File: hw/sch_pcb/I2CDIFF01B.kicad_pcb (KiCad board)
At the start: 2 copper layers, 40.1 x 50.3 mm, 56 parts, among them J1 JUMP_4X2, J10 JUMP_3X2, J11 JUMP2_2x1, J12 CONN_3, J13 JUMP_3X2, J14 JUMP2_2x1, J15 CONN_3, J16 CONN1_1, J17 JUMP2_2x1, J18 CONN1_1, J19 JUMP_2x1, J2 RJ45_RJHSE-5384, J20 JUMP_2x1, J21 JUMP_2x1, J22 JUMP_2x1, J23 JUMP_2x1, J3 JUMP_2x1, J4 JUMP_2x1, J5 JUMP_2x1, J6 JUMP_2x1, J7 JUMP_2x1, J8 JUMP_2x1, J9 JUMP_2x1, M1 HOLE, M2 HOLE, M3 HOLE, M4 HOLE, U1 LM1117 5V, U2 LM1117 3V3, U3 PCA9616

Commit message: Update workflow and KiCAD project to v 9.
Other:
- net class Default removed
- net class dif removed
